File: ATTinyAmpDriver.brd (EAGLE design)
At the start: 30 x 15 mm, 28 parts, among them Q1 SI2301CDS, Q2 BC846, U1 SPX5205M5-L-3-3, U2 ATTINY5-TSHR, U3 MCP6L2-X_SN, X1 DIODES, X2 INPUT

Commit message: Working code and matching board and schematic
Parts:
- R3, R4: value 10k -> 3.9k
- moved C2 11.5 mm to (11.4, 12.9)
- moved R4 11.5 mm to (13.5, 12.9)
- moved R9 10.9 mm to (22.5, 8.05), turned to 90 degrees
- moved R8 9.89 mm to (24.6, 8.05), turned to 270 degrees
- moved C4 8.37 mm to (16.5, 13.3), turned to 0 degrees
- moved R3 3.71 mm to (19.9, 13.4)
- moved R5 2.46 mm to (25.8, 12.9), turned to 0 degrees
- moved X1 1.55 mm to (27.6, 8.26)
- moved Q2 0.15 mm to (20.0, 4.37)
Connections:
- removed net INA+: C4.1, R4.2, U3.3
- removed net VINB-: R8.1, R9.2, U3.6
- new net INA-: R8.1, R9.2, U3.2
- new net INB+: C4.1, R4.2, U3.5
- net D-: now also U3.3; no longer R3.1
- net MEASURE: now also C2.1, U3.6; no longer R9.1
- net OUTA: now also R3.1, R9.1; no longer C2.1, U3.2, U3.5
Routing:
- net INA+: track 8.03 -> 0.00 mm
- net GND: track 7.19 -> 1.25 mm, vias 3 -> 4
- net VINB-: track 5.53 -> 0.00 mm
- net MOSFET: track 16.4 -> 10.9 mm
- net N$8: track 3.75 -> 8.52 mm
- net INB+: track 0.00 -> 4.38 mm
- net INA-: track 0.00 -> 4.20 mm
- net D-: track 8.70 -> 11.7 mm
- net N$3: track 5.58 -> 7.27 mm
- net MEASURE: track 11.1 -> 12.0 mm
- net OUTA: track 10.00 -> 10.7 mm
Other:
- board text added: "EWM 20130630 AT DRIVER 3"
- board text removed: "EWM 20130623 AT DRIVER 3"

Commit message: Added test points around op-amp filter
Parts:
- added MEASURE, OUTA, PWM: TPI, Personal:TPI_PAD
Connections:
- net MEASURE: now also MEASURE.P$1
- net N$5: now also PWM.P$1
- net OUTA: now also OUTA.P$1
Routing:
- net N$5: track 4.03 -> 5.36 mm
- net OUTA: track 10.7 -> 11.7 mm
- net MEASURE: track 12.0 -> 12.8 mm
Changed lines of the file:
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@@
 <attribute name="VALUE" x="22.5806" y="8.9408" size="1.27" layer="27" rot="R270"/>
 </element>
+<element name="PWM" library="Personal" package="TPI_PAD" value="TPI" x="22.0472" y="4.318"/>
+<element name="MEASURE" library="Personal" package="TPI_PAD" value="TPI" x="10.8712" y="6.4008"/>
+<element name="OUTA" library="Personal" package="TPI_PAD" value="TPI" x="20.4216" y="6.6802"/>
 </elements>
 <signals>
@@
 <wire x1="14.6558" y1="10.2362" x2="15.6464" y2="10.2362" width="0.4064" layer="1"/>
 <wire x1="15.6464" y1="10.2362" x2="15.6972" y2="10.1854" width="0.4064" layer="1"/>
+<contactref element="MEASURE" pad="P$1"/>
+<wire x1="10.8712" y1="6.4008" x2="11.684" y2="6.4008" width="0.4064" layer="1"/>
 </signal>
 <signal name="MOSFET">
@@
 <wire x1="19.2786" y1="3.429" x2="19.8804" y2="3.429" width="0.4064" layer="1"/>
 <wire x1="19.8804" y1="3.429" x2="20.0406" y2="3.2688" width="0.4064" layer="1"/>
+<contactref element="PWM" pad="P$1"/>
+<wire x1="22.0472" y1="4.318" x2="21.978" y2="4.318" width="0.4064" layer="1"/>
+<wire x1="21.978" y1="4.318" x2="21.978" y2="3.0582" width="0.4064" layer="1"/>
 </signal>
 <signal name="N$6">
@@
 <wire x1="21.6408" y1="7.2136" x2="22.518" y2="7.2136" width="0.4064" layer="1"/>
 <wire x1="22.518" y1="7.2136" x2="22.5298" y2="7.2018" width="0.4064" layer="1"/>
+<contactref element="OUTA" pad="P$1"/>
+<wire x1="20.4216" y1="6.6802" x2="20.4216" y2="7.6454" width="0.4064" layer="1"/>
 </signal>
 <signal name="N$1">
